Commit message: 1.add xarm base car 2.add some virtual link in xarm for collision avoidance

File: resources/mobile_manipulator/xarm/urdf/xarm6_robot.urdf (robot description, URDF)
Before this commit: robot xarm6, 10 links, 9 joints
Links:
- added link base_car; collision mesh filename=package://ocs2_robotic_assets/resources/mobile_manipulator/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; visual mesh filename=package://ocs2_robotic_assets/resources/mobile_manipulator/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
- added link link5_virtual_1; collision box size=0.01 0.01 0.01; visual box size=0.01 0.01 0.01
- link ee_link: geometry collision box size=0.01 0.01 0.01; visual box size=0.01 0.01 0.01
Joints:
- added joint base_car_joint: type fixed, parent root, child base_car, origin xyz=0 0.0 0.0 rpy=0.0 0.0 0.0
- added joint link5_virtual_1_joint: type fixed, parent link5, child link5_virtual_1, origin xyz=0.038 0.0 0.0 rpy=0.0 0.0 0.0
- joint ee_fixed_joint: origin xyz=0.0 0.0 0.0 rpy=0.0 0.0 1.5707963 -> xyz=0.0 0.0 0.39 rpy=0.0 0.0 1.5707963

Commit message: 将xarm urdf中工具方向调整为与carm_controller中一致

File: resources/mobile_manipulator/xarm/urdf/xarm6_robot.urdf (robot description, URDF)
Before this commit: robot xarm6, 12 links, 11 joints
Joints:
- joint ee_fixed_joint: origin xyz=0.0 0.0 0.39 rpy=0.0 0.0 1.5707963 -> xyz=0.0 0.0 0.39 rpy=0.0 0.0 0.0
